Commit message: assets/prl_ur5: update manually calibrated urdf

File: mime/assets/prl_ur5/robot.urdf (robot description, URDF)
Before this commit: robot prl_ur5_robot, 77 links, 76 joints
Joints:
- joint right_camera_color_optical_joint: origin xyz=0 0 0 rpy=-1.5707963267948966 0 -1.5707963267948966 -> xyz=0 0 0 rpy=-1.5540411677948966 0.001 -1.5607963267948966
