Commit message: assets/prl_ur5: add vention stand model

File: mime/assets/prl_ur5/table.urdf (robot description, URDF)
Before this commit: robot prl_ur5_robot, 3 links, 2 joints
Links:
- link stand_link: geometry collision mesh filename=./meshes/prl_ur5/vention_tower_1.stl; collision mesh filename=./meshes/prl_ur5/vention_tower_2.stl
- link table_link: geometry collision mesh filename=./meshes/prl_ur5/vention_table2.stl; visual mesh filename=./meshes/prl_ur5/vention_table4_decimated6.stl
Joints:
- joint table_fix: parent stand_link -> prl_ur5_base

Commit message: assets: update floor and table urdf

File: mime/assets/prl_ur5/table.urdf (robot description, URDF)
Before this commit: robot prl_ur5_robot, 3 links, 2 joints
Links:
- link stand_link: geometry collision mesh filename=./meshes/prl_ur5/vention_tower_1.stl; collision mesh filename=./meshes/prl_ur5/vention_tower_2.stl
- link table_link: geometry collision mesh filename=./meshes/prl_ur5/vention_table2.stl; visual mesh filename=./meshes/prl_ur5/vention_table4_decimated6.obj
