Commit message: Update all mime to last version

File: mime/assets/prl_ur5/cage_floor.urdf (robot description, URDF)
Before this commit: robot cage.urdf, 1 links, 0 joints
Links:
- added link p1, mass .0; collision box size=0 0 0; visual mesh filename=plane.obj scale=4 3.5 1
Joints:
- added joint j0: type fixed, parent p0, child p1, origin xyz=0.0 0.0 0.0. rpy=0.0 0.0 0.0
